Commit message: Diagnose TurtleBot3 compatibility for TF and odom

File: robot_description/urdf/robot.urdf.xacro (robot description, xacro)
@@ -9,6 +9,8 @@
   <xacro:property name="wheel_y_offset" value="${wheel_separation / 2.0}"/>
   <xacro:property name="wheel_z_offset" value="${wheel_radius}"/>
-  <xacro:property name="scan_z_offset" value="0.105"/>
-  <xacro:property name="imu_z_offset" value="0.060"/>
+  <xacro:property name="scan_x_offset" value="-0.032"/>
+  <xacro:property name="scan_z_offset" value="0.172"/>
+  <xacro:property name="imu_x_offset" value="-0.032"/>
+  <xacro:property name="imu_z_offset" value="0.068"/>
   <xacro:property name="caster_radius" value="0.016"/>
   <xacro:property name="caster_x_offset" value="-0.065"/>
@@ -55,5 +57,5 @@
     <parent link="base_link"/>
     <child link="base_scan"/>
-    <origin xyz="0 0 ${scan_z_offset}" rpy="0 0 0"/>
+    <origin xyz="${scan_x_offset} 0 ${scan_z_offset}" rpy="0 0 0"/>
   </joint>
   <link name="base_scan">
@@ -80,5 +82,5 @@
     <parent link="base_link"/>
     <child link="imu_link"/>
-    <origin xyz="0 0 ${imu_z_offset}" rpy="0 0 0"/>
+    <origin xyz="${imu_x_offset} 0 ${imu_z_offset}" rpy="0 0 0"/>
   </joint>
   <link name="imu_link">

Commit message: Diagnose lidar scan angle indexing and TF wiring

File: robot_description/urdf/robot.urdf.xacro (robot description, xacro)
@@ -1,4 +1,5 @@
 <?xml version="1.0"?>
 <robot xmlns:xacro="http://www.ros.org/wiki/xacro" name="turtlebot3_burger_hw">
+  <xacro:arg name="scan_yaw_offset" default="0.0"/>
   <xacro:property name="base_radius" value="0.089"/>
   <xacro:property name="base_height" value="0.085"/>
@@ -11,4 +12,5 @@
   <xacro:property name="scan_x_offset" value="-0.032"/>
   <xacro:property name="scan_z_offset" value="0.172"/>
+  <xacro:property name="scan_yaw_offset" value="$(arg scan_yaw_offset)"/>
   <xacro:property name="imu_x_offset" value="-0.032"/>
   <xacro:property name="imu_z_offset" value="0.068"/>
@@ -57,5 +59,5 @@
     <parent link="base_link"/>
     <child link="base_scan"/>
-    <origin xyz="${scan_x_offset} 0 ${scan_z_offset}" rpy="0 0 0"/>
+    <origin xyz="${scan_x_offset} 0 ${scan_z_offset}" rpy="0 0 ${scan_yaw_offset}"/>
   </joint>
   <link name="base_scan">

Commit message: Align hardware bringup with TurtleBot3 contract

File: robot_description/urdf/robot.urdf.xacro (robot description, xacro)
@@ -2,12 +2,14 @@
 <robot xmlns:xacro="http://www.ros.org/wiki/xacro" name="turtlebot3_burger_hw">
   <xacro:arg name="scan_yaw_offset" default="0.0"/>
+  <xacro:arg name="namespace" default=""/>
+  <xacro:property name="namespace" value="$(arg namespace)"/>
   <xacro:property name="base_radius" value="0.089"/>
   <xacro:property name="base_height" value="0.085"/>
-  <xacro:property name="base_z" value="0.0335"/>
+  <xacro:property name="base_z" value="0.010"/>
   <xacro:property name="wheel_radius" value="0.033"/>
   <xacro:property name="wheel_width" value="0.018"/>
   <xacro:property name="wheel_separation" value="0.160"/>
   <xacro:property name="wheel_y_offset" value="${wheel_separation / 2.0}"/>
-  <xacro:property name="wheel_z_offset" value="${wheel_radius}"/>
+  <xacro:property name="wheel_z_offset" value="0.023"/>
   <xacro:property name="scan_x_offset" value="-0.032"/>
   <xacro:property name="scan_z_offset" value="0.172"/>
@@ -16,6 +18,6 @@
   <xacro:property name="imu_z_offset" value="0.068"/>
   <xacro:property name="caster_radius" value="0.016"/>
-  <xacro:property name="caster_x_offset" value="-0.065"/>
-  <xacro:property name="caster_z_offset" value="${caster_radius}"/>
+  <xacro:property name="caster_x_offset" value="-0.081"/>
+  <xacro:property name="caster_z_offset" value="-0.004"/>
   <material name="dark_grey">
     <color rgba="0.25 0.25 0.28 1.0"/>
@@ -30,11 +32,11 @@
     <color rgba="0.7 0.7 0.72 1.0"/>
   </material>
-  <link name="base_footprint"/>
-  <joint name="base_footprint_joint" type="fixed">
-    <parent link="base_footprint"/>
-    <child link="base_link"/>
+  <link name="${namespace}base_footprint"/>
+  <joint name="${namespace}base_footprint_joint" type="fixed">
+    <parent link="${namespace}base_footprint"/>
+    <child link="${namespace}base_link"/>
     <origin xyz="0 0 ${base_z}" rpy="0 0 0"/>
   </joint>
-  <link name="base_link">
+  <link name="${namespace}base_link">
     <visual>
       <origin xyz="0 0 0" rpy="0 0 0"/>
@@ -56,10 +58,10 @@
     </inertial>
   </link>
-  <joint name="base_scan_joint" type="fixed">
-    <parent link="base_link"/>
-    <child link="base_scan"/>
+  <joint name="${namespace}base_scan_joint" type="fixed">
+    <parent link="${namespace}base_link"/>
+    <child link="${namespace}base_scan"/>
     <origin xyz="${scan_x_offset} 0 ${scan_z_offset}" rpy="0 0 ${scan_yaw_offset}"/>
   </joint>
-  <link name="base_scan">
+  <link name="${namespace}base_scan">
     <visual>
       <origin xyz="0 0 0" rpy="0 0 0"/>
@@ -81,10 +83,10 @@
     </inertial>
   </link>
-  <joint name="imu_joint" type="fixed">
-    <parent link="base_link"/>
-    <child link="imu_link"/>
+  <joint name="${namespace}imu_joint" type="fixed">
+    <parent link="${namespace}base_link"/>
+    <child link="${namespace}imu_link"/>
     <origin xyz="${imu_x_offset} 0 ${imu_z_offset}" rpy="0 0 0"/>
   </joint>
-  <link name="imu_link">
+  <link name="${namespace}imu_link">
     <visual>
       <origin xyz="0 0 0" rpy="0 0 0"/>
@@ -106,11 +108,11 @@
     </inertial>
   </link>
-  <joint name="wheel_left_joint" type="continuous">
-    <parent link="base_link"/>
-    <child link="left_wheel_link"/>
+  <joint name="${namespace}wheel_left_joint" type="continuous">
+    <parent link="${namespace}base_link"/>
+    <child link="${namespace}wheel_left_link"/>
     <origin xyz="0 ${wheel_y_offset} ${wheel_z_offset}" rpy="-1.57079632679 0 0"/>
     <axis xyz="0 0 1"/>
   </joint>
-  <link name="left_wheel_link">
+  <link name="${namespace}wheel_left_link">
     <visual>
       <origin xyz="0 0 0" rpy="0 0 0"/>
@@ -132,11 +134,11 @@
     </inertial>
   </link>
-  <joint name="wheel_right_joint" type="continuous">
-    <parent link="base_link"/>
-    <child link="right_wheel_link"/>
+  <joint name="${namespace}wheel_right_joint" type="continuous">
+    <parent link="${namespace}base_link"/>
+    <child link="${namespace}wheel_right_link"/>
     <origin xyz="0 -${wheel_y_offset} ${wheel_z_offset}" rpy="-1.57079632679 0 0"/>
     <axis xyz="0 0 1"/>
   </joint>
-  <link name="right_wheel_link">
+  <link name="${namespace}wheel_right_link">
     <visual>
       <origin xyz="0 0 0" rpy="0 0 0"/>
@@ -158,10 +160,10 @@
     </inertial>
   </link>
-  <joint name="caster_back_joint" type="fixed">
-    <parent link="base_link"/>
-    <child link="caster_back_link"/>
-    <origin xyz="${caster_x_offset} 0 ${caster_z_offset}" rpy="0 0 0"/>
+  <joint name="${namespace}caster_back_joint" type="fixed">
+    <parent link="${namespace}base_link"/>
+    <child link="${namespace}caster_back_link"/>
+    <origin xyz="${caster_x_offset} 0 ${caster_z_offset}" rpy="-1.57079632679 0 0"/>
   </joint>
-  <link name="caster_back_link">
+  <link name="${namespace}caster_back_link">
     <visual>
       <origin xyz="0 0 0" rpy="0 0 0"/>

Commit message: Fix robot description TF and mesh integration

File: robot_description/urdf/robot.urdf.xacro (robot description, xacro)
@@ -1,84 +1,157 @@
 <?xml version="1.0"?>
 <robot xmlns:xacro="http://www.ros.org/wiki/xacro" name="turtlebot3_burger_hw">
+  <xacro:arg name="namespace" default=""/>
   <xacro:arg name="scan_yaw_offset" default="0.0"/>
-  <xacro:arg name="namespace" default=""/>
   <xacro:property name="namespace" value="$(arg namespace)"/>
-  <xacro:property name="base_radius" value="0.089"/>
-  <xacro:property name="base_height" value="0.085"/>
-  <xacro:property name="base_z" value="0.010"/>
-  <xacro:property name="wheel_radius" value="0.033"/>
-  <xacro:property name="wheel_width" value="0.018"/>
-  <xacro:property name="wheel_separation" value="0.160"/>
-  <xacro:property name="wheel_y_offset" value="${wheel_separation / 2.0}"/>
-  <xacro:property name="wheel_z_offset" value="0.023"/>
-  <xacro:property name="scan_x_offset" value="-0.032"/>
-  <xacro:property name="scan_z_offset" value="0.172"/>
   <xacro:property name="scan_yaw_offset" value="$(arg scan_yaw_offset)"/>
-  <xacro:property name="imu_x_offset" value="-0.032"/>
-  <xacro:property name="imu_z_offset" value="0.068"/>
-  <xacro:property name="caster_radius" value="0.016"/>
-  <xacro:property name="caster_x_offset" value="-0.081"/>
-  <xacro:property name="caster_z_offset" value="-0.004"/>
-  <material name="dark_grey">
-    <color rgba="0.25 0.25 0.28 1.0"/>
+  <!-- Init colour -->
+  <material name="black">
+    <color rgba="0.0 0.0 0.0 1.0"/>
   </material>
-  <material name="black">
-    <color rgba="0.1 0.1 0.1 1.0"/>
+  <material name="dark">
+    <color rgba="0.3 0.3 0.3 1.0"/>
+  </material>
+  <material name="light_black">
+    <color rgba="0.4 0.4 0.4 1.0"/>
   </material>
   <material name="blue">
-    <color rgba="0.1 0.45 0.85 1.0"/>
+    <color rgba="0.0 0.0 0.8 1.0"/>
   </material>
-  <material name="silver">
-    <color rgba="0.7 0.7 0.72 1.0"/>
+  <material name="green">
+    <color rgba="0.0 0.8 0.0 1.0"/>
+  </material>
+  <material name="grey">
+    <color rgba="0.5 0.5 0.5 1.0"/>
+  </material>
+  <material name="orange">
+    <color rgba="1.0 0.4235 0.0392 1.0"/>
+  </material>
+  <material name="brown">
+    <color rgba="0.8706 0.8118 0.7647 1.0"/>
+  </material>
+  <material name="red">
+    <color rgba="0.8 0.0 0.0 1.0"/>
+  </material>
+  <material name="white">
+    <color rgba="1.0 1.0 1.0 1.0"/>
   </material>
   <link name="${namespace}base_footprint"/>
-  <joint name="${namespace}base_footprint_joint" type="fixed">
+  <joint name="${namespace}base_joint" type="fixed">
     <parent link="${namespace}base_footprint"/>
     <child link="${namespace}base_link"/>
-    <origin xyz="0 0 ${base_z}" rpy="0 0 0"/>
+    <origin xyz="0.0 0.0 0.010" rpy="0 0 0"/>
   </joint>
   <link name="${namespace}base_link">
     <visual>
+      <origin xyz="-0.032 0 0.0" rpy="0 0 0"/>
+      <geometry>
+        <mesh filename="package://robot_description/meshes/bases/burger_base.stl" scale="0.001 0.001 0.001"/>
+      </geometry>
+      <material name="light_black"/>
+    </visual>
+    <collision>
+      <origin xyz="-0.032 0 0.070" rpy="0 0 0"/>
+      <geometry>
+        <box size="0.140 0.140 0.143"/>
+      </geometry>
+    </collision>
+    <inertial>
       <origin xyz="0 0 0" rpy="0 0 0"/>
+      <mass value="8.2573504e-01"/>
+      <inertia
+        ixx="2.2124416e-03"
+        ixy="-1.2294101e-05"
+        ixz="3.4938785e-05"
+        iyy="2.1193702e-03"
+        iyz="-5.0120904e-06"
+        izz="2.0064271e-03"/>
+    </inertial>
+  </link>
+  <joint name="${namespace}wheel_left_joint" type="continuous">
+    <parent link="${namespace}base_link"/>
+    <child link="${namespace}wheel_left_link"/>
+    <origin xyz="0.0 0.08 0.023" rpy="-1.57 0 0"/>
+    <axis xyz="0 0 1"/>
+  </joint>
+  <link name="${namespace}wheel_left_link">
+    <visual>
+      <origin xyz="0 0 0" rpy="1.57 0 0"/>
       <geometry>
-        <cylinder radius="${base_radius}" length="${base_height}"/>
+        <mesh filename="package://robot_description/meshes/wheels/left_tire.stl" scale="0.001 0.001 0.001"/>
       </geometry>
-      <material name="dark_grey"/>
+      <material name="dark"/>
     </visual>
     <collision>
       <origin xyz="0 0 0" rpy="0 0 0"/>
       <geometry>
-        <cylinder radius="${base_radius}" length="${base_height}"/>
+        <cylinder length="0.018" radius="0.033"/>
       </geometry>
     </collision>
     <inertial>
-      <origin xyz="0 0 0" rpy="0 0 0"/>
-      <mass value="1.2"/>
-      <inertia ixx="0.008" ixy="0.0" ixz="0.0" iyy="0.008" iyz="0.0" izz="0.012"/>
+      <origin xyz="0 0 0"/>
+      <mass value="2.8498940e-02"/>
+      <inertia
+        ixx="1.1175580e-05"
+        ixy="-4.2369783e-11"
+        ixz="-5.9381719e-09"
+        iyy="1.1192413e-05"
+        iyz="-1.4400107e-11"
+        izz="2.0712558e-05"/>
     </inertial>
   </link>
-  <joint name="${namespace}base_scan_joint" type="fixed">
+  <joint name="${namespace}wheel_right_joint" type="continuous">
     <parent link="${namespace}base_link"/>
-    <child link="${namespace}base_scan"/>
-    <origin xyz="${scan_x_offset} 0 ${scan_z_offset}" rpy="0 0 ${scan_yaw_offset}"/>
+    <child link="${namespace}wheel_right_link"/>
+    <origin xyz="0.0 -0.080 0.023" rpy="-1.57 0 0"/>
+    <axis xyz="0 0 1"/>
   </joint>
-  <link name="${namespace}base_scan">
+  <link name="${namespace}wheel_right_link">
     <visual>
-      <origin xyz="0 0 0" rpy="0 0 0"/>
+      <origin xyz="0 0 0" rpy="1.57 0 0"/>
       <geometry>
-        <cylinder radius="0.028" length="0.035"/>
+        <mesh filename="package://robot_description/meshes/wheels/right_tire.stl" scale="0.001 0.001 0.001"/>
       </geometry>
-      <material name="blue"/>
+      <material name="dark"/>
     </visual>
     <collision>
       <origin xyz="0 0 0" rpy="0 0 0"/>
       <geometry>
-        <cylinder radius="0.028" length="0.035"/>
+        <cylinder length="0.018" radius="0.033"/>
       </geometry>
     </collision>
     <inertial>
-      <origin xyz="0 0 0" rpy="0 0 0"/>
-      <mass value="0.08"/>
-      <inertia ixx="0.00003" ixy="0.0" ixz="0.0" iyy="0.00003" iyz="0.0" izz="0.00004"/>
+      <origin xyz="0 0 0"/>
+      <mass value="2.8498940e-02"/>
+      <inertia
+        ixx="1.1175580e-05"
+        ixy="-4.2369783e-11"
+        ixz="-5.9381719e-09"
+        iyy="1.1192413e-05"
+        iyz="-1.4400107e-11"
+        izz="2.0712558e-05"/>
+    </inertial>
+  </link>
+  <joint name="${namespace}caster_back_joint" type="fixed">
+    <parent link="${namespace}base_link"/>
+    <child link="${namespace}caster_back_link"/>
+    <origin xyz="-0.081 0 -0.004" rpy="-1.57 0 0"/>
+  </joint>
+  <link name="${namespace}caster_back_link">
+    <collision>
+      <origin xyz="0 0.001 0" rpy="0 0 0"/>
+      <geometry>
+        <box size="0.030 0.009 0.020"/>
+      </geometry>
+    </collision>
+    <inertial>
+      <origin xyz="0 0 0"/>
+      <mass value="0.005"/>
+      <inertia
+        ixx="0.001"
+        ixy="0.0"
+        ixz="0.0"
+        iyy="0.001"
+        iyz="0.0"
+        izz="0.001"/>
     </inertial>
   </link>
@@ -86,101 +159,36 @@
     <parent link="${namespace}base_link"/>
     <child link="${namespace}imu_link"/>
-    <origin xyz="${imu_x_offset} 0 ${imu_z_offset}" rpy="0 0 0"/>
+    <origin xyz="-0.032 0 0.068" rpy="0 0 0"/>
   </joint>
-  <link name="${namespace}imu_link">
+  <link name="${namespace}imu_link"/>
+  <joint name="${namespace}scan_joint" type="fixed">
+    <parent link="${namespace}base_link"/>
+    <child link="${namespace}base_scan"/>
+    <origin xyz="-0.032 0 0.172" rpy="0 0 ${scan_yaw_offset}"/>
+  </joint>
+  <link name="${namespace}base_scan">
     <visual>
-      <origin xyz="0 0 0" rpy="0 0 0"/>
+      <origin xyz="0 0 0.0" rpy="0 0 0"/>
       <geometry>
-        <box size="0.025 0.025 0.010"/>
+        <mesh filename="package://robot_description/meshes/sensors/lds.stl" scale="0.001 0.001 0.001"/>
       </geometry>
-      <material name="silver"/>
+      <material name="dark"/>
     </visual>
     <collision>
-      <origin xyz="0 0 0" rpy="0 0 0"/>
+      <origin xyz="0.015 0 -0.0065" rpy="0 0 0"/>
       <geometry>
-        <box size="0.025 0.025 0.010"/>
+        <cylinder length="0.0315" radius="0.055"/>
       </geometry>
     </collision>
     <inertial>
-      <origin xyz="0 0 0" rpy="0 0 0"/>
-      <mass value="0.02"/>
-      <inertia ixx="0.000002" ixy="0.0" ixz="0.0" iyy="0.000002" iyz="0.0" izz="0.000003"/>
-    </inertial>
-  </link>
-  <joint name="${namespace}wheel_left_joint" type="continuous">
-    <parent link="${namespace}base_link"/>
-    <child link="${namespace}wheel_left_link"/>
-    <origin xyz="0 ${wheel_y_offset} ${wheel_z_offset}" rpy="-1.57079632679 0 0"/>
-    <axis xyz="0 0 1"/>
-  </joint>
-  <link name="${namespace}wheel_left_link">
-    <visual>
-      <origin xyz="0 0 0" rpy="0 0 0"/>
-      <geometry>
-        <cylinder radius="${wheel_radius}" length="${wheel_width}"/>
-      </geometry>
-      <material name="black"/>
-    </visual>
-    <collision>
-      <origin xyz="0 0 0" rpy="0 0 0"/>
-      <geometry>
-        <cylinder radius="${wheel_radius}" length="${wheel_width}"/>
-      </geometry>
-    </collision>
-    <inertial>
-      <origin xyz="0 0 0" rpy="0 0 0"/>
-      <mass value="0.08"/>
-      <inertia ixx="0.00005" ixy="0.0" ixz="0.0" iyy="0.00003" iyz="0.0" izz="0.00003"/>
-    </inertial>
-  </link>
-  <joint name="${namespace}wheel_right_joint" type="continuous">
-    <parent link="${namespace}base_link"/>
-    <child link="${namespace}wheel_right_link"/>
-    <origin xyz="0 -${wheel_y_offset} ${wheel_z_offset}" rpy="-1.57079632679 0 0"/>
-    <axis xyz="0 0 1"/>
-  </joint>
-  <link name="${namespace}wheel_right_link">
-    <visual>
-      <origin xyz="0 0 0" rpy="0 0 0"/>
-      <geometry>
-        <cylinder radius="${wheel_radius}" length="${wheel_width}"/>
-      </geometry>
-      <material name="black"/>
-    </visual>
-    <collision>
-      <origin xyz="0 0 0" rpy="0 0 0"/>
-      <geometry>
-        <cylinder radius="${wheel_radius}" length="${wheel_width}"/>
-      </geometry>
-    </collision>
-    <inertial>
-      <origin xyz="0 0 0" rpy="0 0 0"/>
-      <mass value="0.08"/>
-      <inertia ixx="0.00005" ixy="0.0" ixz="0.0" iyy="0.00003" iyz="0.0" izz="0.00003"/>
-    </inertial>
-  </link>
-  <joint name="${namespace}caster_back_joint" type="fixed">
-    <parent link="${namespace}base_link"/>
-    <child link="${namespace}caster_back_link"/>
-    <origin xyz="${caster_x_offset} 0 ${caster_z_offset}" rpy="-1.57079632679 0 0"/>
-  </joint>
-  <link name="${namespace}caster_back_link">
-    <visual>
-      <origin xyz="0 0 0" rpy="0 0 0"/>
-      <geometry>
-        <sphere radius="${caster_radius}"/>
-      </geometry>
-      <material name="silver"/>
-    </visual>
-    <collision>
-      <origin xyz="0 0 0" rpy="0 0 0"/>
-      <geometry>
-        <sphere radius="${caster_radius}"/>
-      </geometry>
-    </collision>
-    <inertial>
-      <origin xyz="0 0 0" rpy="0 0 0"/>
-      <mass value="0.03"/>
-      <inertia ixx="0.000003" ixy="0.0" ixz="0.0" iyy="0.000003" iyz="0.0" izz="0.000003"/>
+      <mass value="0.114"/>
+      <origin xyz="0 0 0"/>
+      <inertia
+        ixx="0.001"
+        ixy="0.0"
+        ixz="0.0"
+        iyy="0.001"
+        iyz="0.0"
+        izz="0.001"/>
     </inertial>
   </link>
